File: TurtleBoard.brd (EAGLE design)
At the start: 85 x 56 mm, 304 parts, among them IC1 IP101A, IC10 LMV324, IC11 TS482, IC12 AP22802, IC14 ATMEGA32U2-QFN32, IC2 PAM2312A, IC3 XC6SLX25-CSG324, IC4 PAM2312A, IC5 TPD12S521, IC6 PAM2312A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

Commit message: v1.1 As built, Q3 2019
Parts:
- removed R121: 1k5, SEI:0402
- IC12: value AP22802 -> AP22802B
- IC3: value XC6SLX25-CSG324 -> XC6SLX45-2CSG324C
- IC7: value M25P16 -> MX25R3235F; device MC:SO08 -> MC:SOIJ-8
- SK1: value RJ45+MAG+LED-HR911105A -> (none)
- SK5: value USB-SOCKET-MICRO-B -> USB-SOCKET-MICRO-B-PTH; device MC:USB-MICRO-B -> MC:USB-MICRO-B-PTH
- X3: device MC:XTAL-SMD-32X25 -> MC:CRYSTAL-ABM3
- moved SW1 34.8 mm to (45.2, 5.20), turned to 270 degrees
- moved C81 3.60 mm to (45.3, 21.0)
- moved C80 3.60 mm to (45.3, 13.9)
- moved C95 1.66 mm to (18.0, 23.5)
- moved C93 0.90 mm to (6.20, 23.0)
- moved C11 0.90 mm to (17.5, 4.90)
- moved C85 0.80 mm to (46.1, 7.50)
- moved C10 0.80 mm to (15.9, 4.10)
- moved C52 0.80 mm to (35.5, 47.1)
- moved X3 0.51 mm to (14.1, 23.8)
- moved IC7 0.40 mm to (34.5, 45.9), turned to 0 degrees
- moved C47 0.20 mm to (26.2, 32.7)
- moved C83 0.10 mm to (48.6, 14.1)
Connections:
- new net FLASH-SIO2: IC3.T14, IC7.3
- new net FLASH-SIO3: IC3.T6, IC7.7
- new net V: C52.2, IC7.8
- net 3V3: no longer C52.2, IC7.3, IC7.7, IC7.8, R121.2
- net GND: now also SK5.P$3, SK5.P$4
- net GPIO20: now also IC3.U17
- net GPIO21: now also IC3.T18
- net GPIO23: now also IC3.U18
- net N$15: no longer R121.1
- net N$43: now also X3.2; no longer X3.3
Routing:
- net N$85: track 13.7 -> 57.3 mm, vias 2 -> 3
- net GPIO21: track 0.00 -> 38.9 mm, vias 0 -> 1
- net GPIO20: track 0.00 -> 37.0 mm, vias 0 -> 1
- net GPIO23: track 0.00 -> 17.2 mm, vias 0 -> 2
- net FLASH-SIO3: track 0.00 -> 11.6 mm, vias 0 -> 2
- net FLASH-SIO2: track 0.00 -> 8.60 mm, vias 0 -> 2
- net N$74: track 10.0 -> 18.4 mm
- net 3V3: track 81.0 -> 73.7 mm, vias 87 -> 84
- net N$81: track 15.4 -> 21.6 mm
- net V: track 0.00 -> 5.14 mm, vias 0 -> 1
- net GND: track 247.2 -> 251.9 mm, vias 235 -> 233
- net N$25: track 0.00 -> 4.45 mm
- net N$45: track 8.19 -> 11.8 mm
- net N$47: track 7.06 -> 10.3 mm
- net USB_N: track 52.6 -> 50.3 mm
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Other:
- board text added: "1"
- board text added: "RESET"
- board text added: "Turtle Board 1V1 (c) CoreSemi 2019"
- board text removed: "Turtle Board 1V0 (c) SEI 2016"
