File: TurtleBoard.sch (EAGLE design)
At the start: 304 parts, among them IC1 IP101A, IC10 LMV324, IC11 TS482, IC12 AP22802, IC14 ATMEGA32U2-QFN32, IC2 PAM2312A, IC3 XC6SLX25-CSG324, IC4 PAM2312A, IC5 TPD12S521, IC6 PAM2312A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

Commit message: v1.1 As built, Q3 2019
Parts:
- removed R121: 1k5, SEI:R-0402
- IC12: value AP22802 -> AP22802B; PN AP22802AW5-7DICT-ND -> (none)
- IC3: value XC6SLX25-CSG324 -> XC6SLX45-2CSG324C; PN (none) -> 122-1673-ND
- IC7: value M25P16 -> MX25R3235F; device MC:SPI-FLASH-SO8 -> MC:SPI-FLASH-QUADSO8-WIDE; PN M25P16-VME6TGCT-ND -> 1092-1174-ND
- SK1: value RJ45+MAG+LED-HR911105A -> (none)
- SK5: value USB-SOCKET-MICRO-B -> USB-SOCKET-MICRO-B-PTH; device MC:USB-SOCKET-MICRO-B -> MC:USB-SOCKET-MICRO-B-PTH; PN 609-4613-1-ND -> 609-4618-1-ND
- X3: device MC:CRYSTAL-2PIN-32X25 -> MC:CRYSTAL-2PIN-ABM3; PN SER3628CT-ND -> 535-10630-1-ND
Connections:
- new net FLASH-SIO2: IC3-BANK2.IO_L12P_D1_MISO2_2, IC7.!WP/SIO2
- new net FLASH-SIO3: IC3-BANK2.IO_L45P_2, IC7.!RST/SIO3
- new net V: C52.2, IC7.VCC
- net 3V3: no longer C52.2, IC7.!HOLD, IC7.!WP, IC7.VCC, R121.2
- net FLASH-MISO: now also IC7.DO/SIO1; no longer IC7.DO
- net FLASH-MOSI: now also IC7.DI/SIO0; no longer IC7.DI
- net GPIO20: now also IC3-BANK1.IO_L52P_M1DQ14_1
- net GPIO21: now also IC3-BANK1.IO_L51N_M1DQ13_1
- net GPIO23: now also IC3-BANK1.IO_L52N_M1DQ15_1
- net N$15: no longer R121.1
Other:
- moved on the sheet: C52, IC10A, IC10B, IC10C, IC10D, IC7, R47
